File: STM32_boardv2.kicad_pcb (KiCad board)
At the start: 4 copper layers, 124.5 x 84.5 mm, 64 parts, among them J1 Conn_01x02_Pin, J10 Conn_01x02_Pin, J11 Conn_01x02_Pin, J12 Conn_01x06_Pin, J13 Screw_Terminal_01x02, J14 Screw_Terminal_01x02, J15 Screw_Terminal_01x02, J16 Conn_01x02_Pin, J17 Conn_01x02_Pin, J2 Conn_01x09_Pin, J4 Conn_01x09_Pin, J5 Conn_01x04_Pin, J6 Conn_01x03_Pin, J7 USB_B_Micro, J8 Conn_01x04_Pin, J9 Conn_01x02_Pin, SW1 SW_SPDT, SW2 SW_SPDT, SW3 SW_MEC_5G, SW4 SW_SPDT, U1 AMS1117-3.3, U2 AMS1117-3.3, U3 STM32F103C8T6, U4 USBLC6-2SC6, U5 SN74HCT08N, U6 SN74HCT08N, U7 L298N, Y1 16MHz

Commit message: Add files via upload
Parts:
- added G***: LOGO, LOGO, F.Cu at (196.2, 114.5)
- C11, C7: value CALCULATE -> 27p
- C13: value 100n -> 10n
- SW1, SW2, SW4: footprint Button_Switch_SMD:SW_SPDT_PCM12 -> Library:SW_MINI-SPDT-SW
- SW3: footprint Button_Switch_SMD:SW_MEC_5GSH9 -> Library:SW_4-1437565-1
- moved U6 10.3 mm to (174.3, 102.0)
- moved J11 9.11 mm to (182.6, 109.3), turned to -90 degrees
- moved H2 9.05 mm to (202.2, 53.6)
- moved H3 7.99 mm to (202.2, 125.0)
- moved SW3 5.31 mm to (166.4, 91.6), turned to 90 degrees
- moved H4 3.75 mm to (96.7, 125.0)
- moved SW4 3.03 mm to (164.4, 67.5)
- moved U4 3.00 mm to (194.2, 78.2)
- moved R6 2.20 mm to (188.9, 77.2)
- moved J7 1.95 mm to (201.7, 77.8)
- moved SW1 1.20 mm to (155.4, 103.2)
- moved SW2 0.55 mm to (136.6, 122.0)
- moved H1 0.53 mm to (96.7, 53.6)
Routing:
- net Net-(SW2-A): track 0.00 -> 21.4 mm, vias 0 -> 1
- net +5V: track 115.1 -> 101.0 mm, vias 2 -> 0
- net IN3: track 81.1 -> 70.0 mm
- net IN4: track 87.5 -> 76.5 mm
- net U4_1A: track 31.6 -> 42.1 mm
- net U4_1B: track 36.8 -> 46.8 mm
- net VBUS: track 10.6 -> 20.5 mm
- net Net-(J10-Pin_2): track 6.81 -> 15.9 mm
- net GND: track 80.1 -> 87.3 mm, vias 82 -> 81
- net Net-(J11-Pin_1): track 5.90 -> 11.7 mm
- net /SW_BOOT0: track 7.18 -> 12.0 mm
- net /VIN: track 8.99 -> 13.6 mm
- net PA15: track 41.6 -> 45.0 mm
- net Net-(U3-PA3): track 32.2 -> 29.1 mm
- net USB_D-: track 6.89 -> 9.95 mm
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Other:
- board size 124.5 x 84.5 mm -> 115.5 x 81.4 mm
- board text added: "+3.3V"
- board text added: "+5V"
- board text added: "ENA"
- board text added: "ENB"
- board text added: "GND"
- board text added: "IN1"
- board text added: "IN2"
- board text added: "IN3"
- board text added: "IN4"
- board text added: "MISO"
- board text added: "MOSI"
- board text added: "PA10"
- board text added: "PA15"
- board text added: "PA4"
- board text added: "PB0"
- board text added: "PB0_5V"
- board text added: "PB1"
- board text added: "PB12"
- board text added: "PB13"
- board text added: "PB14"
- board text added: "PB15"
- board text added: "PB1_5V"
- board text added: "PB2"
- board text added: "PB3"
- board text added: "PB4"
- board text added: "PB5"
- board text added: "PB8"
- board text added: "PB9"
- board text added: "PC13"
- board text added: "PC14"
- board text added: "PC15"
- board text added: "SCK"
- board text added: "SCL"
- board text added: "SDA"
- board text added: "SWDCLK"
- board text added: "SWDIO"
- board text added: "UART_RX"
- board text added: "UART_TX"
