File: STM32_boardv2.kicad_sch (KiCad schematic)
At the start: 64 parts, among them J1 USB_B_Micro, J10 Conn_01x02_Pin, J11 Conn_01x02_Pin, J12 Conn_01x04_Pin, J13 Screw_Terminal_01x02, J14 Screw_Terminal_01x02, J15 Screw_Terminal_01x02, J2 Conn_01x04_Pin, J4 Conn_01x09_Pin, J5 Conn_01x06_Pin, J6 Conn_01x02_Pin, J7 Conn_01x03_Pin, J8 Conn_01x09_Pin, J9 Conn_01x02_Pin, SW1 SW_MEC_5G, SW1 SW_SPDT, SW2 SW_SPDT, SW4 SW_SPDT, U1 STM32F103C8T6, U2 AMS1117-3.3, U3 SN74HCT08N, U4 SN74HCT08N, U5 AMS1117-3.3, U6 USBLC6-2SC6, U7 L298N, Y1 16MHz

Commit message: Add files via upload
Parts:
- C10, C11: value CALCULATE -> 27p
- C6: value 100n -> 10n
- SW1: footprint Button_Switch_SMD:SW_MEC_5GSH9 -> Library:SW_4-1437565-1
- SW1, SW2, SW4: footprint Button_Switch_SMD:SW_SPDT_PCM12 -> Library:SW_MINI-SPDT-SW
Changed lines of the file:
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@@
       (effects (font (size 1.27 1.27)) (justify left))
     )
-    (property "Footprint" "Button_Switch_SMD:SW_SPDT_PCM12" (at 64.77 101.6 0)
+    (property "Footprint" "Library:SW_MINI-SPDT-SW" (at 64.77 101.6 0)
       (effects (font (size 1.27 1.27)) hide)
     )
@@
       (effects (font (size 1.27 1.27)) (justify left))
     )
-    (property "Value" "CALCULATE" (at 96.52 100.33 0)
+    (property "Value" "27p" (at 96.52 100.33 0)
       (effects (font (size 1.27 1.27)) (justify left))
     )
@@
       (effects (font (size 1.27 1.27)) (justify left))
     )
-    (property "Footprint" "Button_Switch_SMD:SW_SPDT_PCM12" (at 354.33 41.91 0)
+    (property "Footprint" "Library:SW_MINI-SPDT-SW" (at 354.33 41.91 0)
       (effects (font (size 1.27 1.27)) hide)
     )
@@
       (effects (font (size 1.27 1.27)) (justify left))
     )
-    (property "Value" "CALCULATE" (at 118.11 100.33 0)
+    (property "Value" "27p" (at 118.11 100.33 0)
       (effects (font (size 1.27 1.27)) (justify left))
     )
@@
       (effects (font (size 1.27 1.27)) (justify right))
     )
-    (property "Footprint" "Button_Switch_SMD:SW_MEC_5GSH9" (at 72.39 80.01 0)
+    (property "Footprint" "Library:SW_4-1437565-1" (at 72.39 80.01 0)
       (effects (font (size 1.27 1.27)) hide)
     )
@@
       (effects (font (size 1.27 1.27)) (justify left))
     )
-    (property "Footprint" "Button_Switch_SMD:SW_SPDT_PCM12" (at 21.59 100.33 0)
+    (property "Footprint" "Library:SW_MINI-SPDT-SW" (at 21.59 100.33 0)
       (effects (font (size 1.27 1.27)) hide)
     )
@@
       (effects (font (size 1.27 1.27)) (justify left))
     )
-    (property "Value" "100n" (at 171.45 64.77 0)
+    (property "Value" "10n" (at 171.45 64.77 0)
       (effects (font (size 1.27 1.27)) (justify left))
     )
